Commit message: added startup script and set positions

File: tmb_models/urdf/components/rto_blind_parts.urdf.xacro (robot description, xacro)
@@ -80,5 +80,5 @@
                 <origin xyz="0 0 0" rpy="0 0 0"/>
                 <geometry>
-                    <mesh filename="package://tmb_perception/meshes/parts/angle_bracket_usb_hub.dae" scale="${M_SCALE} ${M_SCALE} ${M_SCALE}"/>
+                    <mesh filename="package://tmb_models/meshes/parts/angle_bracket_usb_hub.dae" scale="${M_SCALE} ${M_SCALE} ${M_SCALE}"/>
                 </geometry>
             </visual>
@@ -156,5 +156,5 @@
                 <origin xyz="0 0 0" rpy="0 0 0"/>
                 <geometry>
-                    <mesh filename="package://tmb_perception/meshes/parts/bracket.dae" scale="0.001 ${scale} ${scale}"/>
+                    <mesh filename="package://tmb_models/meshes/parts/bracket.dae" scale="0.001 ${scale} ${scale}"/>
                 </geometry>
                 <material name="red"/>

File: tmb_models/urdf/components/rto_body.urdf.xacro (robot description, xacro)
@@ -20,5 +20,5 @@
                 <origin xyz="0.01 0 0" rpy="0 0 ${M_PI/2}"/>
                 <geometry>
-                    <mesh filename="package://rto_description/meshes/parts/rto_base.dae"
+                    <mesh filename="package://tmb_models/meshes/parts/rto_base.dae"
                         scale="${M_SCALE} ${M_SCALE} ${M_SCALE}"/>
                 </geometry>

File: tmb_models/urdf/components/rto_parts.urdf.xacro (robot description, xacro)
@@ -19,5 +19,5 @@
                 <origin xyz="0 0 0" rpy="0 0 0"/>
                 <geometry>
-                    <mesh filename="package://rto_description/meshes/parts/rto_wheel.dae" scale="${M_SCALE} ${M_SCALE} ${M_SCALE}"/>
+                    <mesh filename="package://tmb_models/meshes/parts/rto_wheel.dae" scale="${M_SCALE} ${M_SCALE} ${M_SCALE}"/>
                 </geometry>
             </visual>
@@ -77,5 +77,5 @@
                 <origin xyz="0 0 0" rpy="0 0 0"/>
                 <geometry>
-                    <mesh filename="package://rto_description/meshes/parts/angle_bracket_usb_hub.dae" scale="${M_SCALE} ${M_SCALE} ${M_SCALE}"/>
+                    <mesh filename="package://tmb_models/meshes/parts/angle_bracket_usb_hub.dae" scale="${M_SCALE} ${M_SCALE} ${M_SCALE}"/>
                 </geometry>
             </visual>
@@ -153,5 +153,5 @@
                 <origin xyz="0 0 0" rpy="0 0 0"/>
                 <geometry>
-                    <mesh filename="package://rto_description/meshes/parts/bracket.dae" scale="0.001 ${scale} ${scale}"/>
+                    <mesh filename="package://tmb_models/meshes/parts/bracket.dae" scale="0.001 ${scale} ${scale}"/>
                 </geometry>
                 <material name="dark_grey"/>

File: tmb_models/urdf/components/rto_platform.urdf (robot description, URDF)
Before this commit: robot rto, 7 links, 6 joints
Links:
- link anglebracketusb_link: geometry visual mesh filename=package://tmb_models/meshes/parts/angle_bracket_usb_hub.dae scale=0.01 0.01 0.01
- link base_link: geometry collision cylinder length=0.05 radius=0.18; visual mesh filename=package://tmb_models/meshes/parts/rto_base.dae scale=0.01 0.01 0.01
- link wheel0_link: geometry visual mesh filename=package://tmb_models/meshes/parts/rto_wheel.dae scale=0.01 0.01 0.01
- link wheel1_link: geometry visual mesh filename=package://tmb_models/meshes/parts/rto_wheel.dae scale=0.01 0.01 0.01
- link wheel2_link: geometry visual mesh filename=package://tmb_models/meshes/parts/rto_wheel.dae scale=0.01 0.01 0.01

File: tmb_models/urdf/components/rto_platform.urdf.xacro (robot description, xacro)
@@ -1,6 +1,6 @@
 <?xml version="1.0"?>
 <robot name="rto" xmlns:xacro="http://wiki.ros.org/xacro">
-    <xacro:include filename="$(find rto_description)/urdf/rto_body.urdf.xacro"/>
-    <xacro:include filename="$(find rto_description)/urdf/rto_parts.urdf.xacro"/>
+    <xacro:include filename="$(find tmb_models)/urdf/rto_body.urdf.xacro"/>
+    <xacro:include filename="$(find tmb_models)/urdf/rto_parts.urdf.xacro"/>
     <xacro:rto_body/>
     <!-- add platform -->

File: tmb_models/urdf/components/rto_platform_kinect.urdf (robot description, URDF)
Before this commit: robot rto, 8 links, 7 joints
Links:
- link anglebracketusb_link: geometry visual mesh filename=package://tmb_models/meshes/parts/angle_bracket_usb_hub.dae scale=0.01 0.01 0.01
- link base_link: geometry collision cylinder length=0.05 radius=0.18; visual mesh filename=package://tmb_models/meshes/parts/rto_base.dae scale=0.01 0.01 0.01
- link kinect_link: geometry collision box size=0.064 0.121 0.0381; visual mesh filename=package://tmb_models/meshes/sensors/kinect.dae
- link wheel0_link: geometry visual mesh filename=package://tmb_models/meshes/parts/rto_wheel.dae scale=0.01 0.01 0.01
- link wheel1_link: geometry visual mesh filename=package://tmb_models/meshes/parts/rto_wheel.dae scale=0.01 0.01 0.01
- link wheel2_link: geometry visual mesh filename=package://tmb_models/meshes/parts/rto_wheel.dae scale=0.01 0.01 0.01

File: tmb_models/urdf/components/rto_platform_kinect.urdf.xacro (robot description, xacro)
@@ -1,7 +1,7 @@
 <?xml version="1.0"?>
 <robot name="rto" xmlns:xacro="http://wiki.ros.org/xacro">
-    <xacro:include filename="$(find rto_description)/urdf/rto_body.urdf.xacro"/>
-    <xacro:include filename="$(find rto_description)/urdf/rto_parts.urdf.xacro"/>
-    <xacro:include filename="$(find rto_description)/urdf/sensors/kinect.urdf.xacro"/>
+    <xacro:include filename="$(find tmb_models)/urdf/rto_body.urdf.xacro"/>
+    <xacro:include filename="$(find tmb_models)/urdf/rto_parts.urdf.xacro"/>
+    <xacro:include filename="$(find tmb_models)/urdf/sensors/kinect.urdf.xacro"/>
     <!-- main rto body -->
     <rto_body/>

File: tmb_models/urdf/robots/rto-1.urdf.xacro (robot description, xacro)
@@ -1,8 +1,8 @@
 <?xml version="1.0"?>
 <robot name="rto" xmlns:xacro="http://wiki.ros.org/xacro">
-  <xacro:include filename="$(find rto_description)/urdf/components/rto_parts.urdf.xacro"/>
-  <xacro:include filename="$(find rto_description)/urdf/components/rto_body.urdf.xacro"/>
-  <xacro:include filename="$(find rto_description)/urdf/sensors/asus_xtion_pro.urdf.xacro"/>
-  <xacro:include filename="$(find rto_description)/urdf/sensors/hokuyo.urdf.xacro"/>
+  <xacro:include filename="$(find tmb_models)/urdf/components/rto_parts.urdf.xacro"/>
+  <xacro:include filename="$(find tmb_models)/urdf/components/rto_body.urdf.xacro"/>
+  <xacro:include filename="$(find tmb_models)/urdf/sensors/asus_xtion_pro.urdf.xacro"/>
+  <xacro:include filename="$(find tmb_models)/urdf/sensors/hokuyo.urdf.xacro"/>
   <xacro:rto_body/>
   <xacro:plate parent="base_link" name="plate"/>
